File: GameClockCircuit/GameClock.kicad_sch (KiCad schematic)
At the start: 0 parts

Commit message: added labelling
Other:
- company: Abhiram Vadali - 2026 -> Abhiram Vadali
- title: Gamified Alarm Clock -> Gamified Alarm Clock - GameClock
Changed lines of the file:
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@@
 	(paper "USLetter")
 	(title_block
-		(title "Gamified Alarm Clock")
+		(title "Gamified Alarm Clock - GameClock")
 		(date "2026-05-11")
 		(rev "1.0")
-		(company "Abhiram Vadali - 2026")
+		(company "Abhiram Vadali")
+		(comment 1 "ATMega328p ")
+		(comment 2 "2026")
+		(comment 3 "**for lack of a better name, it's GameClock")
 	)
 	(sheet_instances
